Commit message: feat: add joint position limits and soft gravity compensation support
This commit adds joint position limit support to the robotic arm system:
1. Add joint lower/upper limit fields to JointConfig and load from YAML config
2. Add SetJointLimit interface to IMotor and implement for DMMotor
3. Add position limit checking and motor stop logic in DMMotor
4. Update URDF joint limits to match config values
5. Add soft limit parameters and force feedback handling to gravity controller
6. Flip auto_reset flag in launch config to True
7. Refactor collision detection method naming convention

File: config/arm.urdf (robot description, URDF)
Before this commit: robot arm, 7 links, 6 joints
Links:
- added link link7, mass 0.060
Joints:
- added joint joint7: type revolute, parent link6, child link7, origin xyz=0.084 0 -0.035 rpy=0 0 0, axis 1 0 0, limit lower=-3.15 upper=3.15 effort=0 velocity=0
- joint joint1: limit lower=-3.14 upper=3.14 effort=0 velocity=0 -> lower=-4 upper=4 effort=0 velocity=0
- joint joint2: limit lower=-3.14 upper=3.14 effort=0 velocity=0 -> lower=-3.14 upper=1.57 effort=0 velocity=0
- joint joint3: limit lower=-3.14 upper=3.14 effort=0 velocity=0 -> lower=-1.57 upper=1.57 effort=0 velocity=0
- joint joint4: limit lower=-3.14 upper=3.14 effort=0 velocity=0 -> lower=-4 upper=4 effort=0 velocity=0
- joint joint5: limit lower=-3.14 upper=3.14 effort=0 velocity=0 -> lower=-2 upper=2 effort=0 velocity=0
- joint joint6: limit lower=-3.15 upper=3.15 effort=0 velocity=0 -> lower=-4 upper=4 effort=0 velocity=0
