Commit message: phase 1.5: connect gazebo ros2 control

File: config/arm.urdf (robot description, URDF)
Before this commit: robot arm, 8 links, 7 joints
Links:
- removed link link7
Joints:
- removed joint joint7
- joint joint1: limit lower=-4 upper=4 effort=0 velocity=0 -> lower=-3.14 upper=3.14 effort=20 velocity=2.0
- joint joint2: limit lower=-3.14 upper=1.57 effort=0 velocity=0 -> lower=-3.14 upper=3.14 effort=20 velocity=2.0
- joint joint3: limit lower=-1.57 upper=1.57 effort=0 velocity=0 -> lower=-3.14 upper=3.14 effort=20 velocity=2.0
- joint joint4: limit lower=-4 upper=4 effort=0 velocity=0 -> lower=-3.14 upper=3.14 effort=20 velocity=2.0
- joint joint5: limit lower=-2 upper=2 effort=0 velocity=0 -> lower=-3.14 upper=3.14 effort=20 velocity=2.0
- joint joint6: limit lower=-4 upper=4 effort=0 velocity=0 -> lower=-3.15 upper=3.15 effort=20 velocity=2.0

File: config/arm_with_d435i.urdf.xacro (robot description, xacro)
@@ -7,6 +7,9 @@
   <xacro:arg name="camera_rpy" default="0 0 0"/>
   <xacro:arg name="camera_use_nominal_extrinsics" default="true"/>
+  <xacro:arg name="use_ros2_control" default="true"/>
+  <xacro:arg name="fix_base_to_world" default="true"/>
   <xacro:include filename="$(find manipulator)/arm.urdf"/>
   <xacro:include filename="$(find manipulator)/sensors/d435i_mount.xacro"/>
+  <xacro:include filename="$(find manipulator)/sensors/gazebo_ros2_control.xacro"/>
   <xacro:windylab_d435i_mount
       camera_enabled="$(arg camera_enabled)"
@@ -16,3 +19,6 @@
       camera_rpy="$(arg camera_rpy)"
       camera_use_nominal_extrinsics="$(arg camera_use_nominal_extrinsics)"/>
+  <xacro:windylab_gazebo_ros2_control
+      use_ros2_control="$(arg use_ros2_control)"
+      fix_base_to_world="$(arg fix_base_to_world)"/>
 </robot>
