Commit message: phase 3: add d435i imu gazebo output

File: config/arm_with_d435i.urdf.xacro (robot description, xacro)
@@ -18,4 +18,13 @@
   <xacro:arg name="rgbd_far" default="5.0"/>
   <xacro:arg name="rgbd_visualize" default="false"/>
+  <xacro:arg name="imu_enabled" default="true"/>
+  <xacro:arg name="imu_namespace" default="d435i"/>
+  <xacro:arg name="imu_topic" default="imu"/>
+  <xacro:arg name="imu_frame_name" default="camera_accel_optical_frame"/>
+  <xacro:arg name="imu_update_rate" default="200"/>
+  <xacro:arg name="imu_visualize" default="false"/>
+  <xacro:arg name="imu_noise_mean" default="0.0"/>
+  <xacro:arg name="imu_angular_velocity_noise_stddev" default="0.0"/>
+  <xacro:arg name="imu_linear_acceleration_noise_stddev" default="0.0"/>
   <xacro:arg name="use_ros2_control" default="true"/>
   <xacro:arg name="fix_base_to_world" default="true"/>
@@ -44,4 +53,15 @@
       rgbd_far="$(arg rgbd_far)"
       rgbd_visualize="$(arg rgbd_visualize)"/>
+  <xacro:windylab_d435i_gazebo_imu
+      imu_enabled="$(arg imu_enabled)"
+      camera_name="$(arg camera_name)"
+      imu_namespace="$(arg imu_namespace)"
+      imu_topic="$(arg imu_topic)"
+      imu_frame_name="$(arg imu_frame_name)"
+      imu_update_rate="$(arg imu_update_rate)"
+      imu_visualize="$(arg imu_visualize)"
+      imu_noise_mean="$(arg imu_noise_mean)"
+      imu_angular_velocity_noise_stddev="$(arg imu_angular_velocity_noise_stddev)"
+      imu_linear_acceleration_noise_stddev="$(arg imu_linear_acceleration_noise_stddev)"/>
   <xacro:windylab_gazebo_ros2_control
       use_ros2_control="$(arg use_ros2_control)"

File: config/sensors/d435i_gazebo.xacro (robot description, xacro)
@@ -53,3 +53,74 @@
     </xacro:if>
   </xacro:macro>
+  <xacro:macro name="windylab_d435i_gazebo_imu"
+      params="imu_enabled:=true
+              camera_name:=camera
+              imu_namespace:=d435i
+              imu_topic:=imu
+              imu_frame_name:=camera_accel_optical_frame
+              imu_update_rate:=200
+              imu_visualize:=false
+              imu_noise_mean:=0.0
+              imu_angular_velocity_noise_stddev:=0.0
+              imu_linear_acceleration_noise_stddev:=0.0">
+    <xacro:if value="${imu_enabled}">
+      <gazebo reference="${camera_name}_link">
+        <sensor type="imu" name="${camera_name}_imu_sensor">
+          <always_on>true</always_on>
+          <update_rate>${imu_update_rate}</update_rate>
+          <visualize>${imu_visualize}</visualize>
+          <imu>
+            <angular_velocity>
+              <x>
+                <noise type="gaussian">
+                  <mean>${imu_noise_mean}</mean>
+                  <stddev>${imu_angular_velocity_noise_stddev}</stddev>
+                </noise>
+              </x>
+              <y>
+                <noise type="gaussian">
+                  <mean>${imu_noise_mean}</mean>
+                  <stddev>${imu_angular_velocity_noise_stddev}</stddev>
+                </noise>
+              </y>
+              <z>
+                <noise type="gaussian">
+                  <mean>${imu_noise_mean}</mean>
+                  <stddev>${imu_angular_velocity_noise_stddev}</stddev>
+                </noise>
+              </z>
+            </angular_velocity>
+            <linear_acceleration>
+              <x>
+                <noise type="gaussian">
+                  <mean>${imu_noise_mean}</mean>
+                  <stddev>${imu_linear_acceleration_noise_stddev}</stddev>
+                </noise>
+              </x>
+              <y>
+                <noise type="gaussian">
+                  <mean>${imu_noise_mean}</mean>
+                  <stddev>${imu_linear_acceleration_noise_stddev}</stddev>
+                </noise>
+              </y>
+              <z>
+                <noise type="gaussian">
+                  <mean>${imu_noise_mean}</mean>
+                  <stddev>${imu_linear_acceleration_noise_stddev}</stddev>
+                </noise>
+              </z>
+            </linear_acceleration>
+          </imu>
+          <plugin name="${camera_name}_imu_controller" filename="libgazebo_ros_imu_sensor.so">
+            <ros>
+              <namespace>${imu_namespace}</namespace>
+              <remapping>~/out:=${imu_topic}</remapping>
+            </ros>
+            <frame_name>${imu_frame_name}</frame_name>
+            <initial_orientation_as_reference>false</initial_orientation_as_reference>
+          </plugin>
+        </sensor>
+      </gazebo>
+    </xacro:if>
+  </xacro:macro>
 </robot>

Commit message: phase 4: parameterize d435i mount mode

File: config/arm_with_d435i.urdf.xacro (robot description, xacro)
@@ -2,8 +2,9 @@
 <robot name="arm" xmlns:xacro="http://www.ros.org/wiki/xacro">
   <xacro:arg name="camera_enabled" default="true"/>
+  <xacro:arg name="camera_mount_mode" default="ee"/>
   <xacro:arg name="camera_name" default="camera"/>
-  <xacro:arg name="camera_parent_link" default="link6"/>
-  <xacro:arg name="camera_xyz" default="0.06 0 0.04"/>
-  <xacro:arg name="camera_rpy" default="0 0 0"/>
+  <xacro:arg name="camera_parent_link" default="auto"/>
+  <xacro:arg name="camera_xyz" default="auto"/>
+  <xacro:arg name="camera_rpy" default="auto"/>
   <xacro:arg name="camera_use_nominal_extrinsics" default="true"/>
   <xacro:arg name="rgbd_enabled" default="true"/>
@@ -33,10 +34,20 @@
   <xacro:include filename="$(find manipulator)/sensors/d435i_gazebo.xacro"/>
   <xacro:include filename="$(find manipulator)/sensors/gazebo_ros2_control.xacro"/>
+  <xacro:property name="camera_mount_mode_arg" value="$(arg camera_mount_mode)"/>
+  <xacro:property name="camera_parent_link_arg" value="$(arg camera_parent_link)"/>
+  <xacro:property name="camera_xyz_arg" value="$(arg camera_xyz)"/>
+  <xacro:property name="camera_rpy_arg" value="$(arg camera_rpy)"/>
+  <xacro:property name="resolved_camera_parent_link"
+                  value="${'base_link' if camera_parent_link_arg == 'auto' and camera_mount_mode_arg == 'base' else 'link6' if camera_parent_link_arg == 'auto' else camera_parent_link_arg}"/>
+  <xacro:property name="resolved_camera_xyz"
+                  value="${'0.12 0 0.36' if camera_xyz_arg == 'auto' and camera_mount_mode_arg == 'base' else '0.06 0 0.04' if camera_xyz_arg == 'auto' else camera_xyz_arg}"/>
+  <xacro:property name="resolved_camera_rpy"
+                  value="${'0 0 0' if camera_rpy_arg == 'auto' else camera_rpy_arg}"/>
   <xacro:windylab_d435i_mount
       camera_enabled="$(arg camera_enabled)"
       camera_name="$(arg camera_name)"
-      camera_parent_link="$(arg camera_parent_link)"
-      camera_xyz="$(arg camera_xyz)"
-      camera_rpy="$(arg camera_rpy)"
+      camera_parent_link="${resolved_camera_parent_link}"
+      camera_xyz="${resolved_camera_xyz}"
+      camera_rpy="${resolved_camera_rpy}"
       camera_use_nominal_extrinsics="$(arg camera_use_nominal_extrinsics)"/>
   <xacro:windylab_d435i_gazebo_rgbd
