Commit message: phase 3 fix: add physical dynamics control mode

File: config/sensors/gazebo_ros2_control.xacro (robot description, xacro)
@@ -42,8 +42,12 @@
           <plugin>gazebo_ros2_control/GazeboSystem</plugin>
         </hardware>
-        <xacro:macro name="windylab_position_joint" params="joint_name lower upper">
+        <xacro:macro name="windylab_controlled_joint" params="joint_name lower upper">
           <joint name="${joint_name}">
             <command_interface name="position">
               <param name="min">${lower}</param>
+              <param name="max">${upper}</param>
+            </command_interface>
+            <command_interface name="velocity">
+              <param name="min">-${upper}</param>
               <param name="max">${upper}</param>
             </command_interface>
@@ -53,10 +57,10 @@
           </joint>
         </xacro:macro>
-        <xacro:windylab_position_joint joint_name="joint1" lower="-3.14" upper="3.14"/>
-        <xacro:windylab_position_joint joint_name="joint2" lower="-3.14" upper="3.14"/>
-        <xacro:windylab_position_joint joint_name="joint3" lower="-3.14" upper="3.14"/>
-        <xacro:windylab_position_joint joint_name="joint4" lower="-3.14" upper="3.14"/>
-        <xacro:windylab_position_joint joint_name="joint5" lower="-3.14" upper="3.14"/>
-        <xacro:windylab_position_joint joint_name="joint6" lower="-3.15" upper="3.15"/>
+        <xacro:windylab_controlled_joint joint_name="joint1" lower="-3.14" upper="3.14"/>
+        <xacro:windylab_controlled_joint joint_name="joint2" lower="-3.14" upper="3.14"/>
+        <xacro:windylab_controlled_joint joint_name="joint3" lower="-3.14" upper="3.14"/>
+        <xacro:windylab_controlled_joint joint_name="joint4" lower="-3.14" upper="3.14"/>
+        <xacro:windylab_controlled_joint joint_name="joint5" lower="-3.14" upper="3.14"/>
+        <xacro:windylab_controlled_joint joint_name="joint6" lower="-3.15" upper="3.15"/>
       </ros2_control>
       <gazebo>
